Commit message: Modified the URDF file and added sample codes for serial communication with arduino

File: robot.urdf (robot description, URDF)
Before this commit: robot simple_arm, 7 links, 6 joints
Links:
- removed link gripper
- removed link link1
- removed link link2
- removed link link3
- removed link link4
- removed link link5
- added link arm1; visual cylinder length=0.13 radius=0.022
- added link arm2; visual cylinder length=0.13 radius=0.011
- added link arm3; visual cylinder length=0.13 radius=0.022
- added link base_rot; visual box size=0.08 0.08 0.1
- added link gripper_link; visual box size=0.1 0.1 0.01
- added link left_finger; visual box size=0.01 0.01 0.05
- added link right_finger; visual box size=0.01 0.01 0.05
- link base_link: geometry visual box size=0.14 0.14 0.08
Joints:
- removed joint joint1
- removed joint joint2
- removed joint joint3
- removed joint joint4
- removed joint joint5
- removed joint joint6
- added joint base_joint: type revolute, parent base_link, child base_rot, origin xyz=0 0 0.1 rpy=0 0 0, axis 0 0 -1, limit lower=0 upper=3.1416 effort=1.0 velocity=1.0
- added joint elbow_joint: type revolute, parent arm1, child arm2, origin xyz=0 0 0.13 rpy=0 0 0, axis 1 0 0, limit lower=-1.3 upper=1.92
- added joint gripper_rotation: type revolute, parent arm3, child gripper_link, origin xyz=0 0 0.13 rpy=0 0 0, axis 0 0 1, limit lower=-1.57 upper=1.57 effort=1.0 velocity=1.0
- added joint left_finger_joint: type prismatic, parent gripper_link, child left_finger, origin xyz=0.025 0 0.025 rpy=0 0 0, axis 1 0 0, limit lower=-0.05 upper=0.0 effort=10.0 velocity=0.1
- added joint right_finger_joint: type prismatic, parent gripper_link, child right_finger, origin xyz=-0.025 0 0.025 rpy=0 0 0, axis -1 0 0, limit lower=-0.05 upper=0.0 effort=10.0 velocity=0.1
- added joint shoulder_joint: type revolute, parent base_rot, child arm1, origin xyz=0 0 0.027 rpy=0 0 0, axis 1 0 0, limit lower=0 upper=1.57
- added joint wrist_joint: type revolute, parent arm2, child arm3, origin xyz=0 0 0.13 rpy=0 0 0, axis 1 0 0, limit lower=-1.3 upper=1.92

Commit message: ...

File: robot.urdf (robot description, URDF)
Before this commit: robot robot_arm, 8 links, 7 joints
Links:
- link arm1: geometry visual cylinder length=0.105 radius=0.013
- link arm2: geometry visual cylinder length=0.126 radius=0.008
- link arm3: geometry visual cylinder length=0.053 radius=0.022
- link base_link: geometry visual box size=0.09 0.09 0.03
- link base_rot: geometry visual box size=0.02 0.04 0.046
- link gripper_link: geometry visual box size=0.002 0.002 0.002
- link left_finger: geometry visual box size=0.01 0.01 0.
Joints:
- joint elbow_joint: origin xyz=0 0 0.13 rpy=0 0 0 -> xyz=0 0 0.126 rpy=0 0 0
- joint gripper_rotation: origin xyz=0 0 0.13 rpy=0 0 0 -> xyz=0 0 0.002 rpy=0 0 0
- joint shoulder_joint: origin xyz=0 0 0.027 rpy=0 0 0 -> xyz=0 0 0.105 rpy=0 0 0
- joint wrist_joint: origin xyz=0 0 0.13 rpy=0 0 0 -> xyz=0 0 0.053 rpy=0 0 0

Commit message: edited the urdf

File: robot.urdf (robot description, URDF)
Before this commit: robot robot_arm, 8 links, 7 joints
Links:
- link left_finger: geometry visual box size=0.003 0.003 0.109
- link right_finger: geometry visual box size=0.003 0.003 0.109

Commit message: trial and error for urdf

File: robot.urdf (robot description, URDF)
Before this commit: robot robot_arm, 8 links, 7 joints
Links:
- link gripper_link: geometry visual box size=0.05 0.05 0.01
- link left_finger: geometry visual box size=0.01 0.01 0.05
- link right_finger: geometry visual box size=0.01 0.01 0.05
Joints:
- removed joint right_finger_joint
- added joint right_finger_fixed: type fixed, parent gripper_link, child right_finger, origin xyz=-0.015 0 0 rpy=0 0 0
- joint base_joint: origin xyz=0 0 0.1 rpy=0 0 0 -> xyz=0 0 0.03 rpy=0 0 0
- joint elbow_joint: origin xyz=0 0 0.126 rpy=0 0 0 -> xyz=0 0 0.105 rpy=0 0 0
- joint gripper_rotation: origin xyz=0 0 0.002 rpy=0 0 0 -> xyz=0 0 0.053 rpy=0 0 0
- joint left_finger_joint: limit lower=-0.05 upper=0.0 effort=10.0 velocity=0.1 -> lower=-0.02 upper=0.02 effort=10.0 velocity=0.1; origin xyz=0.025 0 0.025 rpy=0 0 0 -> xyz=0.015 0 0 rpy=0 0 0
- joint shoulder_joint: limit lower=0 upper=1.57 -> lower=-1.57 upper=1.57; origin xyz=0 0 0.105 rpy=0 0 0 -> xyz=0 0 0.046 rpy=0 0 0
- joint wrist_joint: origin xyz=0 0 0.053 rpy=0 0 0 -> xyz=0 0 0.126 rpy=0 0 0
